File: UPDI_plus_UART/20250807_updi.kicad_pcb (KiCad board)
At the start: 2 copper layers, 53 x 20 mm, 29 parts, among them J1 USB_C_Receptacle_USB2.0_16P, J2 Conn_01x02_Pin, J3 Conn_01x02_Pin, J4 Conn_01x02_Pin, J5 Conn_01x02_Pin, J6 Conn_01x03_Socket, J7 Conn_01x03_Pin, J8 Conn_01x03_Socket, U1 CH342K, U2 AP1117-33

Commit message: Add files via upload
cleaned up schematics and added LCSC part numbers
Parts:
- D4: value LED -> LED Y
- D5: value LED -> LED G
- D6: value LED -> LED B
- D7: value LED -> LED R
- U2: value AP1117-33 -> AMS1117-33
